File: LTPowerAnalyzer_BNC_Adapter/LTPowerAnalyzer_BNC_Adapter.kicad_pcb (KiCad board)
At the start: 2 copper layers, 1 part, among them J1 HTSW-210-08-T-S-RA

Commit message: Major update
Parts:
- added G***: LOGO, spencer-connectors:LTPowerAnalyzerConnections, F.Cu at (146.6, 91.0)
- added GND: TestPoint, TestPoint:TestPoint_Pad_1.5x1.5mm, F.Cu at (186.1, 121.0)
- added J1: 031-5431, SamacSys_Parts:0315431, F.Cu at (106.6, 63.0)
- added J2: 031-5431, SamacSys_Parts:0315431, F.Cu at (106.6, 83.0)
- added J3: 031-5431, SamacSys_Parts:0315431, F.Cu at (106.6, 103.0)
- added J4: 031-5431, SamacSys_Parts:0315431, F.Cu at (106.6, 123.0)
- added R1: 0Ω, Resistor_SMD:R_0805_2012Metric, F.Cu at (183.6, 110.5)
- added W1: TestPoint, TestPoint:TestPoint_Pad_1.5x1.5mm, F.Cu at (186.6, 63.0)
- moved J5 104.5 mm to (189.1, 90.5)
- renumbered J1 to J5
Connections:
- J5 pad 01: unconnected-(J1-Pad01) -> /W1
- J5 pad 02: unconnected-(J1-Pad02) -> /T+
- J5 pad 03: unconnected-(J1-Pad03) -> /T-
- J5 pad 04: unconnected-(J1-Pad04) -> /OUT+
- J5 pad 05: unconnected-(J1-Pad05) -> /OUT-
- J5 pad 06: unconnected-(J1-Pad06) -> /IN+
- J5 pad 07: unconnected-(J1-Pad07) -> /IN-
- J5 pad 08: unconnected-(J1-Pad08) -> /VO+
- J5 pad 09: unconnected-(J1-Pad09) -> /VO-
- J5 pad 10: unconnected-(J1-Pad10) -> GND
Routing:
- net /VO-: track 0.00 -> 92.1 mm
- net /VO+: track 0.00 -> 88.8 mm
- net /T-: track 0.00 -> 85.7 mm
- net /IN+: track 0.00 -> 84.7 mm
- net /IN-: track 0.00 -> 84.7 mm
- net /T+: track 0.00 -> 83.8 mm
- net /OUT-: track 0.00 -> 81.6 mm
- net /OUT+: track 0.00 -> 81.6 mm
- net /W1: track 0.00 -> 4.75 mm
- net GND: track 0.00 -> 3.50 mm
- added copper zone on B.Cu, net GND
- added copper zone on F.Cu, net GND
- added copper zone on In1.Cu, net GND
- added copper zone on In2.Cu, net GND
Other:
- board outline added: 96.5 x 77.5 mm
- copper layers 2 -> 4
- board text added: "IN+/IN-"
- board text added: "OUT+/OUT1"
- board text added: "T+/T-"
- board text added: "VO+/VO-"

Commit message: routing
Routing:
- net GND: track 3.50 -> 11.2 mm
- net /VO-: track 92.1 -> 93.0 mm
- removed copper zone on In1.Cu, net GND
- removed copper zone on In2.Cu, net GND
Other:
- copper layers 4 -> 2

Commit message: updates
Parts:
- J1, J2, J3, J4: footprint SamacSys_Parts:0315431 -> user_footprints:0315431
- renumbered W1 to TP1, GND to TP2
Other:
- board text added: "VOUT+/VOUT-"
- board text removed: "VO+/VO-"
Changed lines of the file:
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@@
 		(descr "SMD rectangular pad as test Point, square 1.5mm side length")
 		(tags "test point SMD pad rectangle square")
-		(property "Reference" "W1"
+		(property "Reference" "TP1"
 			(at 1.955 -0.146801 0)
 			(layer "F.SilkS")
@@
 		(embedded_fonts no)
 	)
-	(footprint "SamacSys_Parts:0315431"
+	(footprint "user_footprints:0315431"
 		(layer "F.Cu")
 		(at 106.646801 82.955 90)
@@
 		(tags "Connector")
 		(property "Reference" "J2"
-			(at 0 -15.675 90)
+			(at 9.455 1.353199 0)
 			(layer "F.SilkS")
 			(effects
@@
 		)
 		(embedded_fonts no)
-		(model "C:\\Code\\gitRepos\\PCB-Projects\\Common\\libs\\SamacSys_Parts.3dshapes\\031-5431.stp"
+		(model "${USER_3DMODELS}/031-5431.stp"
 			(offset
-				(xyz 0 31.06999923 8.060000299)
+				(xyz 0 31 8.2)
 			)
 			(scale
@@
 			)
 			(rotate
-				(xyz -90 0 90)
+				(xyz -90 -0 90)
 			)
 		)
@@
 		(descr "SMD rectangular pad as test Point, square 1.5mm side length")
 		(tags "test point SMD pad rectangle square")
-		(property "Reference" "GND"
+		(property "Reference" "TP2"
 			(at -2.545 -0.146801 0)
 			(layer "F.SilkS")
@@
 		(embedded_fonts no)
 	)
-	(footprint "SamacSys_Parts:0315431"
+	(footprint "user_footprints:0315431"
 		(layer "F.Cu")
 		(at 106.646801 122.955 90)
@@
 		(tags "Connector")
 		(property "Reference" "J4"
-			(at 0 -15.675 90)
+			(at 8.455 4.353199 180)
 			(layer "F.SilkS")
 			(effects
@@
 		)
 		(embedded_fonts no)
-		(model "C:\\Code\\gitRepos\\PCB-Projects\\Common\\libs\\SamacSys_Parts.3dshapes\\031-5431.stp"
+		(model "${USER_3DMODELS}/031-5431.stp"
 			(offset
-				(xyz 0 31.06999923 8.060000299)
+				(xyz 0 31 8.2)
 			)
 			(scale
@@
 			)
 			(rotate
-				(xyz -90 0 90)
+				(xyz -90 -0 90)
 			)
 		)
@@
 		(embedded_fonts no)
 	)
-	(footprint "SamacSys_Parts:0315431"
+	(footprint "user_footprints:0315431"
 		(layer "F.Cu")
 		(at 106.646801 62.955 90)
@@
 		(tags "Connector")
 		(property "Reference" "J1"
-			(at 0 -15.675 90)
+			(at 7.955 4.353199 180)
 			(layer "F.SilkS")
 			(effects
@@
 		)
 		(embedded_fonts no)
-		(model "C:\\Code\\gitRepos\\PCB-Projects\\Common\\libs\\SamacSys_Parts.3dshapes\\031-5431.stp"
+		(model "${USER_3DMODELS}/031-5431.stp"
 			(offset
-				(xyz 0 31.06999923 8.060000299)
+				(xyz 0 31 8.2)
 			)
 			(scale
@@
 			)
 			(rotate
-				(xyz -90 0 90)
+				(xyz -90 -0 90)
 			)
 		)
 	)
-	(footprint "SamacSys_Parts:0315431"
+	(footprint "user_footprints:0315431"
 		(layer "F.Cu")
 		(at 106.646801 102.955 90)
@@
 		(tags "Connector")
 		(property "Reference" "J3"
-			(at 0 -15.675 90)
+			(at 7.455 4.353199 0)
 			(layer "F.SilkS")
 			(effects
@@
 		)
 		(embedded_fonts no)
-		(model "C:\\Code\\gitRepos\\PCB-Projects\\Common\\libs\\SamacSys_Parts.3dshapes\\031-5431.stp"
+		(model "${USER_3DMODELS}/031-5431.stp"
 			(offset
-				(xyz 0 31.06999923 8.060000299)
+				(xyz 0 31 8.2)
 			)
 			(scale
@@
 			)
 			(rotate
-				(xyz -90 0 90)
+				(xyz -90 -0 90)
 			)
 		)
@@
 	)
 	(gr_text "T+/T-"
-		(at 86.051563 53.955 0)
+		(at 110.5 60 0)
 		(layer "F.SilkS")
 		(effects
@@
 	)
 	(gr_text "OUT+/OUT1"
-		(at 82.146801 74.121667 0)
+		(at 112.5 91.5 90)
 		(layer "F.SilkS")
 		(effects
@@
 		)
 	)
-	(gr_text "VO+/VO-"
-		(at 83.765849 114.455 0)
+	(gr_text "VOUT+/VOUT-"
+		(at 110.5 128 0)
 		(layer "F.SilkS")
 		(effects
@@
 	)
 	(gr_text "IN+/IN-"
-		(at 84.527754 94.288333 0)
+		(at 110.5 108.5 0)
 		(layer "F.SilkS")
 		(effects
