File: LTPowerAnalyzer_BNC_Adapter/LTPowerAnalyzer_BNC_Adapter.kicad_sch (KiCad schematic)
At the start: 8 parts, among them J1 HTSW-210-08-T-S-RA, J6 031-5431, J7 031-5431, J8 031-5431, J9 031-5431

Commit message: updates
Parts:
- J1: renamed from J6; footprint 0315431 -> user_footprints:0315431
- J2: renamed from J7; footprint 0315431 -> user_footprints:0315431
- J3: renamed from J8; footprint 0315431 -> user_footprints:0315431
- J4: renamed from J9; footprint 0315431 -> user_footprints:0315431
- renumbered J1 to J5
Changed lines of the file:
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@@
 		(on_board yes)
 		(dnp no)
-		(property "Reference" "J7"
+		(property "Reference" "J2"
 			(at 50.038 65.786 0)
 			(effects
@@
 			)
 		)
-		(property "Footprint" "0315431"
+		(property "Footprint" "user_footprints:0315431"
 			(at 39.37 -32.69 0)
 			(effects
@@
 			(project "LTPowerAnalyzer_BNC_Adapter"
 				(path "/e2208708-0263-4261-ba55-a7849cd966f0"
-					(reference "J7")
+					(reference "J2")
 					(unit 1)
 				)
@@
 		(on_board yes)
 		(dnp no)
-		(property "Reference" "J8"
+		(property "Reference" "J3"
 			(at 50.038 81.026 0)
 			(effects
@@
 			)
 		)
-		(property "Footprint" "0315431"
+		(property "Footprint" "user_footprints:0315431"
 			(at 39.37 -17.45 0)
 			(effects
@@
 			(project "LTPowerAnalyzer_BNC_Adapter"
 				(path "/e2208708-0263-4261-ba55-a7849cd966f0"
-					(reference "J8")
+					(reference "J3")
 					(unit 1)
 				)
@@
 		(on_board yes)
 		(dnp no)
-		(property "Reference" "J9"
+		(property "Reference" "J4"
 			(at 50.038 97.536 0)
 			(effects
@@
 			)
 		)
-		(property "Footprint" "0315431"
+		(property "Footprint" "user_footprints:0315431"
 			(at 39.37 -0.94 0)
 			(effects
@@
 			(project "LTPowerAnalyzer_BNC_Adapter"
 				(path "/e2208708-0263-4261-ba55-a7849cd966f0"
-					(reference "J9")
+					(reference "J4")
 					(unit 1)
 				)
@@
 		(on_board yes)
 		(dnp no)
-		(property "Reference" "J6"
+		(property "Reference" "J1"
 			(at 50.038 50.546 0)
 			(effects
@@
 			)
 		)
-		(property "Footprint" "0315431"
+		(property "Footprint" "user_footprints:0315431"
 			(at 39.37 -47.93 0)
 			(effects
@@
 			(project ""
 				(path "/e2208708-0263-4261-ba55-a7849cd966f0"
-					(reference "J6")
+					(reference "J1")
 					(unit 1)
 				)
@@
 		(on_board yes)
 		(dnp no)
-		(property "Reference" "J1"
+		(property "Reference" "J5"
 			(at 159.004 71.12 0)
 			(effects
@@
 			(project ""
 				(path "/e2208708-0263-4261-ba55-a7849cd966f0"
-					(reference "J1")
+					(reference "J5")
 					(unit 1)
 				)
